File: redox/pcb/rev2.0_ng/kicad_files/redox_rev2_ng.sch (KiCad schematic (older format))
At the start: 147 parts, among them J2 OLED-SSD1306, K1 KEYSW, K10 KEYSW, K11 KEYSW, K12 KEYSW, K13 KEYSW, K14 KEYSW, K15 KEYSW, K16 KEYSW, K17 KEYSW, K18 KEYSW, K19 KEYSW, K2 KEYSW, K20 KEYSW, K21 KEYSW, K22 KEYSW, K23 KEYSW, K24 KEYSW, K25 KEYSW, K26 KEYSW, K27 KEYSW, K28 KEYSW, K29 KEYSW, K3 KEYSW, K30 KEYSW, K31 KEYSW, K32 KEYSW, K33 KEYSW, K34 KEYSW, K35 KEYSW, K4 KEYSW, K5 KEYSW, K6 KEYSW, K7 KEYSW, K8 KEYSW, K9 KEYSW, P1 TC2030-AVR, Q1 2N7002, U1 PRTR5V0U2X, U2 ATmega32U4, Y1 16Mhz

Commit message: Replace the reset switch footprint by something easier to find - 6x6 push button
Parts:
- RST_SW1: footprint redox_footprints:TACT_SWITCH_TVBP06 -> redox_footprints:SW_PUSH_6mm_h4.3mm
Changed lines of the file:
@@
 F 0 "RST_SW1" H 1475 1460 50  0000 C CNN
 F 1 "SW_PUSH" H 1325 1270 50  0000 C CNN
-F 2 "redox_footprints:TACT_SWITCH_TVBP06" H 1325 1350 60  0001 C CNN
+F 2 "redox_footprints:SW_PUSH_6mm_h4.3mm" H 1325 1350 60  0001 C CNN
 F 3 "" H 1325 1350 60  0000 C CNN
 	1    1325 1350
